Commit message: to add simulink model

File: urdf/iiwa7/iiwa7.urdf (robot description, URDF)
Before this commit: robot iiwa7, 9 links, 8 joints
Joints:
- joint iiwa_joint_1: limit lower=-2.96705972839 upper=2.96705972839 effort=300 velocity=10 -> lower=-12.96705972839 upper=12.96705972839 effort=300 velocity=10
- joint iiwa_joint_2: limit lower=-2.09439510239 upper=2.09439510239 effort=300 velocity=10 -> lower=-12.09439510239 upper=12.09439510239 effort=300 velocity=10
- joint iiwa_joint_3: limit lower=-2.96705972839 upper=2.96705972839 effort=300 velocity=10 -> lower=-12.96705972839 upper=12.96705972839 effort=300 velocity=10
- joint iiwa_joint_4: limit lower=-2.09439510239 upper=2.09439510239 effort=300 velocity=10 -> lower=-12.09439510239 upper=12.09439510239 effort=300 velocity=10
- joint iiwa_joint_5: limit lower=-2.96705972839 upper=2.96705972839 effort=300 velocity=10 -> lower=-12.96705972839 upper=12.96705972839 effort=300 velocity=10
- joint iiwa_joint_6: limit lower=-2.09439510239 upper=2.09439510239 effort=300 velocity=10 -> lower=-12.09439510239 upper=12.09439510239 effort=300 velocity=10
- joint iiwa_joint_7: limit lower=-3.05432619099 upper=3.05432619099 effort=300 velocity=10 -> lower=-13.05432619099 upper=13.05432619099 effort=300 velocity=10
