Commit message: update IP urdf

File: urdf/IP/urdf/IP.urdf (robot description, URDF)
Before this commit: robot IP, 4 links, 3 joints
Links:
- removed link link1
- removed link world
- added link car, mass 1; visual mesh filename=package://IP/meshes/link1.STL
- link rod: geometry visual scale value=1
Joints:
- removed joint base_joint
- joint joint1: child link1 -> car
- joint joint2: parent link1 -> car
